File: led-controller-wrover32/led-controller-wrover32.sch (KiCad schematic (older format))
At the start: 40 parts, among them J1 Micro_SD_Card, J2 Conn_01x12, J3 USB_B_Micro, J4 Conn_01x12, J5 Conn_01x04 DNS, J6 Conn_01x02 DNS, J7 Conn_01x02 DNS, J8 Conn_01x04 DNS, Q1 MMBT2222A-TP, Q2 MMBT2222A-TP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

Commit message: Revision 1.1.1, moved things around a little.
Parts:
- removed U5: TPS3809, TO_SOT_Packages_SMD:SOT-23, symbol TI_Power_Supervisor:TPS3809
- J2, J4: footprint aaron:BM12B-SURS-TF -> aaron:BM12B-SRSS-TB
Connections:
- wire segments 230 -> 225
Changed lines of the file:
@@
-$EndComp
-$Comp
-L switch_tact_smt:SW_SPST_KMR2 SW1
-U 1 1 5B95DB65
-P 4500 1600
-F 0 "SW1" V 4540 1459 42  0000 R CNN
-F 1 "KMR2" V 4461 1459 42  0000 R CNN
-F 2 "aaron:SW_SPST_KMR2" H 4500 1600 50  0001 C CNN
-F 3 "" H 4500 1600 50  0001 C CNN
-	1    4500 1600
-	0    -1   -1   0
 $EndComp
 $Comp
@@
 	4500 2100 4500 1800
 Wire Wire Line
-	4500 1800 4600 1800
-Connection ~ 4500 1800
-Wire Wire Line
 	4500 900  4500 800
 Wire Wire Line
 	4950 1700 4950 1800
-Wire Wire Line
-	4950 1800 4600 1800
-Connection ~ 4600 1800
 $Comp
 L Connector:USB_B_Micro J3
@@
 Wire Wire Line
 	4500 1200 4500 1400
-Wire Wire Line
-	4600 1400 4500 1400
-Connection ~ 4500 1400
-Wire Wire Line
-	4600 1400 4950 1400
-Connection ~ 4600 1400
 Connection ~ 4950 1400
 Text Label 4700 6800 0    50   ~ 0
@@
 Wire Wire Line
 	4250 6700 4850 6700
-Wire Wire Line
-	4850 6700 4850 6750
 Text Label 4700 6700 0    50   ~ 0
 DO
@@
 F 0 "J4" H 5570 6567 50  0000 C CNN
 F 1 "Conn_01x12" H 5570 6476 50  0000 C CNN
-F 2 "aaron:BM12B-SURS-TF" H 5650 5850 50  0001 C CNN
+F 2 "aaron:BM12B-SRSS-TB" H 5650 5850 50  0001 C CNN
 F 3 "~" H 5650 5850 50  0001 C CNN
 	1    5650 5850
@@
 Text Label 8000 3050 0    50   ~ 0
 IO27
-$Comp
-L TI_Power_Supervisor:TPS3809 U5
-U 1 1 5BBE98E4
-P 3700 2000
-F 0 "U5" H 3700 2365 50  0000 C CNN
-F 1 "TPS3809" H 3700 2274 50  0000 C CNN
-F 2 "TO_SOT_Packages_SMD:SOT-23" H 3700 2000 50  0001 C CNN
-F 3 "https://media.digikey.com/pdf/Data%20Sheets/Texas%20Instruments%20PDFs/TPS3809xxx-Q1.pdf" H 3700 2000 50  0001 C CNN
-	1    3700 2000
-	1    0    0    -1
-$EndComp
-Wire Wire Line
-	3100 1900 3300 1900
-Wire Wire Line
-	3300 2100 3300 2200
-Wire Wire Line
-	3300 2200 3100 2200
-Wire Wire Line
-	4100 2000 4350 2000
-Text Label 4100 2000 0    50   ~ 0
-RESET
 Wire Wire Line
 	5750 2150 5650 2150
@@
 F 0 "J2" H 3970 7617 50  0000 C CNN
 F 1 "Conn_01x12" H 3970 7526 50  0000 C CNN
-F 2 "aaron:BM12B-SURS-TF" H 4050 6900 50  0001 C CNN
+F 2 "aaron:BM12B-SRSS-TB" H 4050 6900 50  0001 C CNN
 F 3 "~" H 4050 6900 50  0001 C CNN
 	1    4050 6900
 	-1   0    0    -1
 $EndComp
+Wire Wire Line
+	4600 1400 4950 1400
+Wire Wire Line
+	4600 1400 4500 1400
+Connection ~ 4600 1400
+Wire Wire Line
+	4950 1800 4600 1800
+Wire Wire Line
+	4500 1800 4600 1800
+Connection ~ 4600 1800
+Connection ~ 4500 1400
+Connection ~ 4500 1800
+$Comp
+L switch_tact_smt:SW_SPST_KMR2 SW1
+U 1 1 5B95DB65
+P 4500 1600
+F 0 "SW1" V 4540 1459 42  0000 R CNN
+F 1 "KMR2" V 4461 1459 42  0000 R CNN
+F 2 "aaron:SW_SPST_KMR2" H 4500 1600 50  0001 C CNN
+F 3 "" H 4500 1600 50  0001 C CNN
+	1    4500 1600
+	0    -1   -1   0
+$EndComp
 $EndSCHEMATC

Commit message: - Added some more I/O pins to J4 and added pull-up resistors to IO21,   IO22 and IO23. - Cleaned up Torex buck converter - Minor layout changes - Added more ground vias near the antenna. - Added another filter cap for J8 - Added another pin to J8 for +3.3v
Signed-off-by: Aaron Williams <aaron.w2@gmail.com>
Parts:
- removed J8: Conn_01x04 DNS, Pin_Headers:Pin_Header_Straight_1x04_Pitch1.27mm, symbol Connector_Generic:Conn_01x04
- added C15: 1uF 10V, Capacitors_SMD:C_0603, symbol Device:C
- added J8: Conn_01x05, Pin_Headers:Pin_Header_Straight_1x05_Pitch1.27mm, symbol Connector:Conn_01x05
- added R7, R8, R9: 10K, Resistors_SMD:R_0603, symbol Device:R
Connections:
- wire segments 225 -> 240

Commit message: Did some more trace cleanup.
Signed-off-by: Aaron Williams <aaron.w2@gmail.com>
Connections:
- net labels added: USB_D+, USB_D-
Changed lines of the file:
@@
 L Device:C C12
 U 1 1 5BDD8725
-P 5500 4400
-F 0 "C12" H 5615 4446 50  0000 L CNN
-F 1 "10uF 10V" H 5550 4550 50  0000 L CNN
-F 2 "Capacitors_SMD:C_0805" H 5538 4250 50  0001 C CNN
-F 3 "~" H 5500 4400 50  0001 C CNN
-	1    5500 4400
+P 5850 4000
+F 0 "C12" H 5965 4046 50  0000 L CNN
+F 1 "10uF 10V" H 5900 4150 50  0000 L CNN
+F 2 "Capacitors_SMD:C_0805" H 5888 3850 50  0001 C CNN
+F 3 "~" H 5850 4000 50  0001 C CNN
+	1    5850 4000
 	1    0    0    -1
 $EndComp
@@
 L power:GND #PWR033
 U 1 1 5BDD88E3
-P 5500 4750
-F 0 "#PWR033" H 5500 4500 50  0001 C CNN
-F 1 "GND" H 5505 4577 50  0000 C CNN
-F 2 "" H 5500 4750 50  0001 C CNN
-F 3 "" H 5500 4750 50  0001 C CNN
-	1    5500 4750
+P 5850 4350
+F 0 "#PWR033" H 5850 4100 50  0001 C CNN
+F 1 "GND" H 5855 4177 50  0000 C CNN
+F 2 "" H 5850 4350 50  0001 C CNN
+F 3 "" H 5850 4350 50  0001 C CNN
+	1    5850 4350
 	1    0    0    -1
 $EndComp
@@
 L power:+3.3V #PWR032
 U 1 1 5BDD8932
-P 5500 4100
-F 0 "#PWR032" H 5500 3950 50  0001 C CNN
-F 1 "+3.3V" H 5515 4273 50  0000 C CNN
-F 2 "" H 5500 4100 50  0001 C CNN
-F 3 "" H 5500 4100 50  0001 C CNN
-	1    5500 4100
-	1    0    0    -1
-$EndComp
-Wire Wire Line
-	5500 4100 5500 4250
-Wire Wire Line
-	5500 4550 5500 4750
-Text Notes 5550 4550 0    50   ~ 0
+P 5850 3700
+F 0 "#PWR032" H 5850 3550 50  0001 C CNN
+F 1 "+3.3V" H 5865 3873 50  0000 C CNN
+F 2 "" H 5850 3700 50  0001 C CNN
+F 3 "" H 5850 3700 50  0001 C CNN
+	1    5850 3700
+	1    0    0    -1
+$EndComp
+Wire Wire Line
+	5850 3700 5850 3850
+Wire Wire Line
+	5850 4150 5850 4350
+Text Notes 5900 4150 0    50   ~ 0
 Place near ESP32
 Wire Wire Line
@@
 $EndComp
 Wire Wire Line
-	8500 5100 8500 5200
+	8950 5100 8950 5200
 Wire Wire Line
 	8500 5200 8400 5200
@@
 L power:+3.3V #PWR0103
 U 1 1 5BAE6DE9
-P 8500 5100
-F 0 "#PWR0103" H 8500 4950 50  0001 C CNN
-F 1 "+3.3V" H 8400 5250 50  0000 C CNN
-F 2 "" H 8500 5100 50  0001 C CNN
-F 3 "" H 8500 5100 50  0001 C CNN
-	1    8500 5100
+P 8950 5100
+F 0 "#PWR0103" H 8950 4950 50  0001 C CNN
+F 1 "+3.3V" H 8950 5250 50  0000 C CNN
+F 2 "" H 8950 5100 50  0001 C CNN
+F 3 "" H 8950 5100 50  0001 C CNN
+	1    8950 5100
 	1    0    0    -1
 $EndComp
@@
 P 8950 5500
 F 0 "C15" H 9065 5546 50  0000 L CNN
-F 1 "1uF 10V" H 8650 5750 50  0000 L CNN
+F 1 "1uF 10V" H 9000 5650 50  0000 L CNN
 F 2 "Capacitors_SMD:C_0603" H 8988 5350 50  0001 C CNN
 F 3 "~" H 8950 5500 50  0001 C CNN
@@
 Wire Wire Line
 	6600 6150 6600 6550
+Connection ~ 8950 5200
+Text Label 6250 2250 0    50   ~ 0
+USB_D+
+Text Label 6250 2350 0    50   ~ 0
+USB_D-
 $EndSCHEMATC

Commit message: Fixed several issues.
1. GPIOs 16 and 17 should not be connected.
2. GPIO 35 was mislabeled GPIO36.  It's input only and would not have
   been able to drive the TS pin oin the MAX chip.
3. Routed GPIO35 to J4.
4. Added a 0.1uF bypass capacitor for Wrover32 like the datasheet recommends.
5. Added another 3.3v pin to J4 after removing GPIOs 16 and 17.

Signed-off-by: Aaron Williams <aaron.w2@gmail.com>
Parts:
- added C16: 1uF 10V, Capacitors_SMD:C_0603, symbol Device:C
Connections:
- net labels added: IO35
- net labels removed: IO16, IO17, IO36
- wire segments 240 -> 242
Changed lines of the file:
@@
 Text Label 6800 4150 0    50   ~ 0
 IO33_H
-Text Label 6800 3650 0    50   ~ 0
-IO36
 Wire Wire Line
 	3750 5250 3200 5250
@@
 IO15
 Wire Wire Line
-	3750 4350 3200 4350
-Text Label 3200 4350 0    50   ~ 0
-IO16
-Wire Wire Line
-	3750 4450 3200 4450
-Text Label 3200 4450 0    50   ~ 0
-IO17
-Wire Wire Line
 	3750 4550 3200 4550
 Text Label 3200 4550 0    50   ~ 0
@@
 	3750 5650 3200 5650
 Text Label 3200 5650 0    50   ~ 0
-IO36
+IO35
 Wire Wire Line
 	2800 3950 3750 3950
@@
 Text Label 6350 5650 0    50   ~ 0
 IO5
-Wire Wire Line
-	5850 5750 6450 5750
-Text Label 6300 5750 0    50   ~ 0
-IO17
-Wire Wire Line
-	5850 5850 6450 5850
-Text Label 6300 5850 0    50   ~ 0
-IO16
 Text Label 4600 6900 0    50   ~ 0
 IO33_H
@@
 	8950 5350 8950 5200
 Wire Wire Line
-	6700 5050 6700 5950
-Wire Wire Line
 	5850 5950 6700 5950
 Wire Wire Line
@@
 Text Label 6250 2350 0    50   ~ 0
 USB_D-
+Wire Wire Line
+	5850 5850 6700 5850
+Connection ~ 6700 5850
+Wire Wire Line
+	6700 5850 6700 5950
+$Comp
+L power:+3.3V #PWR0107
+U 1 1 5BD2AFEE
+P 6800 3500
+F 0 "#PWR0107" H 6800 3350 50  0001 C CNN
+F 1 "+3.3V" H 6815 3673 50  0000 C CNN
+F 2 "" H 6800 3500 50  0001 C CNN
+F 3 "" H 6800 3500 50  0001 C CNN
+	1    6800 3500
+	1    0    0    -1
+$EndComp
+Wire Wire Line
+	6800 3500 6800 3650
+$Comp
+L Device:C C16
+U 1 1 5BD3CD62
+P 6250 4000
+F 0 "C16" H 6365 4046 50  0000 L CNN
+F 1 "1uF 10V" H 5950 4250 50  0000 L CNN
+F 2 "Capacitors_SMD:C_0603" H 6288 3850 50  0001 C CNN
+F 3 "~" H 6250 4000 50  0001 C CNN
+	1    6250 4000
+	1    0    0    -1
+$EndComp
+Wire Wire Line
+	6250 3850 5850 3850
+Connection ~ 5850 3850
+Wire Wire Line
+	5850 4150 6250 4150
+Connection ~ 5850 4150
+Wire Wire Line
+	6700 5050 6700 5850
+Wire Wire Line
+	5850 5750 6450 5750
+Text Label 6300 5750 0    50   ~ 0
+IO35
 $EndSCHEMATC

Commit message: Added microphone and updated README
Signed-off-by: Aaron Williams <aaron.w2@gmail.com>
Parts:
- added MIC1: SPH0645LM4H-B, digikey-footprints:SPH0645LM4H-B, symbol dk_Microphones:SPH0645LM4H-B
- added R10: 100K, Resistors_SMD:R_0603, symbol Device:R
Connections:
- wire segments 242 -> 247
Changed lines of the file:
@@
 L power:VBUS #PWR012
 U 1 1 5B9E5410
-P 4550 6350
-F 0 "#PWR012" H 4550 6200 50  0001 C CNN
-F 1 "VBUS" H 4565 6523 50  0000 C CNN
-F 2 "" H 4550 6350 50  0001 C CNN
-F 3 "" H 4550 6350 50  0001 C CNN
-	1    4550 6350
-	1    0    0    -1
-$EndComp
-Wire Wire Line
-	4250 6400 4550 6400
+P 4200 6550
+F 0 "#PWR012" H 4200 6400 50  0001 C CNN
+F 1 "VBUS" H 4215 6723 50  0000 C CNN
+F 2 "" H 4200 6550 50  0001 C CNN
+F 3 "" H 4200 6550 50  0001 C CNN
+	1    4200 6550
+	1    0    0    -1
+$EndComp
+Wire Wire Line
+	3900 6600 4200 6600
 $Comp
 L power:+3.3V #PWR013
 U 1 1 5B9E8C3A
-P 4850 6400
-F 0 "#PWR013" H 4850 6250 50  0001 C CNN
-F 1 "+3.3V" H 4865 6573 50  0000 C CNN
-F 2 "" H 4850 6400 50  0001 C CNN
-F 3 "" H 4850 6400 50  0001 C CNN
-	1    4850 6400
+P 4500 6600
+F 0 "#PWR013" H 4500 6450 50  0001 C CNN
+F 1 "+3.3V" H 4515 6773 50  0000 C CNN
+F 2 "" H 4500 6600 50  0001 C CNN
+F 3 "" H 4500 6600 50  0001 C CNN
+	1    4500 6600
 	1    0    0    -1
 $EndComp
@@
 L power:GND #PWR016
 U 1 1 5B9EC681
-P 5050 6600
-F 0 "#PWR016" H 5050 6350 50  0001 C CNN
-F 1 "GND" H 5055 6427 50  0000 C CNN
-F 2 "" H 5050 6600 50  0001 C CNN
-F 3 "" H 5050 6600 50  0001 C CNN
-	1    5050 6600
+P 4700 6800
+F 0 "#PWR016" H 4700 6550 50  0001 C CNN
+F 1 "GND" H 4705 6627 50  0000 C CNN
+F 2 "" H 4700 6800 50  0001 C CNN
+F 3 "" H 4700 6800 50  0001 C CNN
+	1    4700 6800
 	1    0    0    -1
 $EndComp
@@
 	650  6150 650  6300
 Wire Wire Line
-	4250 6800 4850 6800
-Wire Wire Line
-	4250 6900 4850 6900
-Wire Wire Line
-	4250 7000 4850 7000
-Wire Wire Line
-	4250 7100 4850 7100
-Wire Wire Line
-	4250 7200 4850 7200
+	3900 7000 4500 7000
+Wire Wire Line
+	3900 7100 4500 7100
+Wire Wire Line
+	3900 7200 4500 7200
+Wire Wire Line
+	3900 7300 4500 7300
+Wire Wire Line
+	3900 7400 4500 7400
 $Comp
 L Device:R_Pack04 RN2
@@
 	4500 1200 4500 1400
 Connection ~ 4950 1400
-Text Label 4700 6800 0    50   ~ 0
+Text Label 4350 7000 0    50   ~ 0
 IO34
 Text Label 6300 5350 0    50   ~ 0
@@
 Text Label 6350 5650 0    50   ~ 0
 IO5
-Text Label 4600 6900 0    50   ~ 0
+Text Label 4250 7100 0    50   ~ 0
 IO33_H
-Text Label 4600 7000 0    50   ~ 0
+Text Label 4250 7200 0    50   ~ 0
 IO32_H
-Text Label 4600 7100 0    50   ~ 0
+Text Label 4250 7300 0    50   ~ 0
 IO26_H
-Text Label 4600 7200 0    50   ~ 0
+Text Label 4250 7400 0    50   ~ 0
 IO25_H
 $Comp
@@
 IO27
 Wire Wire Line
-	4250 6700 4850 6700
-Text Label 4700 6700 0    50   ~ 0
+	3900 6900 4500 6900
+Text Label 4350 6900 0    50   ~ 0
 DO
 $Comp
@@
 	5850 6250 6800 6250
 Wire Wire Line
-	4250 7400 4850 7400
-Wire Wire Line
-	4250 7500 4850 7500
-Wire Wire Line
-	4250 7300 4850 7300
-Text Label 4600 7500 0    50   ~ 0
+	3900 7600 4500 7600
+Wire Wire Line
+	3900 7700 4500 7700
+Wire Wire Line
+	3900 7500 4500 7500
+Text Label 4250 7700 0    50   ~ 0
 RESET
-Text Label 4450 7300 0    50   ~ 0
+Text Label 4100 7500 0    50   ~ 0
 SENSOR_VN
-Text Label 4450 7400 0    50   ~ 0
+Text Label 4100 7600 0    50   ~ 0
 SENSOR_VP
 Wire Wire Line
@@
 $EndComp
 Wire Wire Line
-	4250 6600 4850 6600
-Wire Wire Line
-	4850 6400 4850 6600
-Wire Wire Line
-	5050 6600 5050 6500
-Wire Wire Line
-	5050 6500 4250 6500
+	3900 6800 4500 6800
+Wire Wire Line
+	4500 6600 4500 6800
+Wire Wire Line
+	4700 6800 4700 6700
+Wire Wire Line
+	4700 6700 3900 6700
 Text Label 7850 2600 0    50   ~ 0
 IO27
@@
 Connection ~ 5650 2050
 Wire Wire Line
-	4550 6400 4550 6350
+	4200 6600 4200 6550
 $Comp
 L Connector_Generic:Conn_01x12 J2
 U 1 1 5B9D440B
-P 4050 6900
-F 0 "J2" H 3970 7617 50  0000 C CNN
-F 1 "Conn_01x12" H 3970 7526 50  0000 C CNN
-F 2 "aaron:BM12B-SRSS-TB" H 4050 6900 50  0001 C CNN
-F 3 "~" H 4050 6900 50  0001 C CNN
-	1    4050 6900
+P 3700 7100
+F 0 "J2" H 3620 7817 50  0000 C CNN
+F 1 "Conn_01x12" H 3620 7726 50  0000 C CNN
+F 2 "aaron:BM12B-SRSS-TB" H 3700 7100 50  0001 C CNN
+F 3 "~" H 3700 7100 50  0001 C CNN
+	1    3700 7100
 	-1   0    0    -1
 $EndComp
@@
 Text Label 6300 5750 0    50   ~ 0
 IO35
+$Comp
+L dk_Microphones:SPH0645LM4H-B MIC1
+U 1 1 5BD7F7C7
+P 5400 7200
+F 0 "MIC1" H 5841 7253 60  0000 L CNN
+F 1 "SPH0645LM4H-B" H 5841 7147 60  0000 L CNN
+F 2 "digikey-footprints:SPH0645LM4H-B" H 5600 7400 60  0001 L CNN
+F 3 "http://www.knowles.com/eng/content/download/5988/105771/version/4/file/SPH0645LM4H-BRevB.PDF" H 5600 7500 60  0001 L CNN
+F 4 "423-1405-1-ND" H 5600 7600 60  0001 L CNN "Digi-Key_PN"
+F 5 "SPH0645LM4H-B" H 5600 7700 60  0001 L CNN "MPN"
+F 6 "Audio Products" H 5600 7800 60  0001 L CNN "Category"
+F 7 "Microphones" H 5600 7900 60  0001 L CNN "Family"
+F 8 "http://www.knowles.com/eng/content/download/5988/105771/version/4/file/SPH0645LM4H-BRevB.PDF" H 5600 8000 60  0001 L CNN "DK_Datasheet_Link"
+F 9 "/product-detail/en/knowles/SPH0645LM4H-B/423-1405-1-ND/5332432" H 5600 8100 60  0001 L CNN "DK_Detail_Page"
+F 10 "MIC MEMS DIGITAL I2S OMNI -26DB" H 5600 8200 60  0001 L CNN "Description"
+F 11 "Knowles" H 5600 8300 60  0001 L CNN "Manufacturer"
+F 12 "Active" H 5600 8400 60  0001 L CNN "Status"
+	1    5400 7200
+	1    0    0    -1
+$EndComp
+$Comp
+L power:+3.3V #PWR040
+U 1 1 5BD90296
+P 5400 6800
+F 0 "#PWR040" H 5400 6650 50  0001 C CNN
+F 1 "+3.3V" H 5300 6950 50  0000 C CNN
+F 2 "" H 5400 6800 50  0001 C CNN
+F 3 "" H 5400 6800 50  0001 C CNN
+	1    5400 6800
+	1    0    0    -1
+$EndComp
+$Comp
+L power:GND #PWR043
+U 1 1 5BD90301
+P 5400 7600
+F 0 "#PWR043" H 5400 7350 50  0001 C CNN
+F 1 "GND" H 5405 7427 50  0000 C CNN
+F 2 "" H 5400 7600 50  0001 C CNN
+F 3 "" H 5400 7600 50  0001 C CNN
+	1    5400 7600
+	1    0    0    -1
+$EndComp
+$Comp
+L power:GND #PWR041
+U 1 1 5BD9074D
+P 4650 7500
+F 0 "#PWR041" H 4650 7250 50  0001 C CNN
+F 1 "GND" H 4655 7327 50  0000 C CNN
+F 2 "" H 4650 7500 50  0001 C CNN
+F 3 "" H 4650 7500 50  0001 C CNN
+	1    4650 7500
+	1    0    0    -1
+$EndComp
+Wire Wire Line
+	4650 7500 4650 7200
+Wire Wire Line
+	4650 7200 5000 7200
+$Comp
+L Device:R R10
+U 1 1 5BDB1170
+P 5800 7350
+F 0 "R10" V 5850 7500 50  0000 C CNN
+F 1 "100K" V 5800 7350 50  0000 C CNN
+F 2 "Resistors_SMD:R_0603" V 5730 7350 50  0001 C CNN
+F 3 "~" H 5800 7350 50  0001 C CNN
+	1    5800 7350
+	-1   0    0    1
+$EndComp
+$Comp
+L power:GND #PWR042
+U 1 1 5BDB12F7
+P 5800 7500
+F 0 "#PWR042" H 5800 7250 50  0001 C CNN
+F 1 "GND" H 5805 7327 50  0000 C CNN
+F 2 "" H 5800 7500 50  0001 C CNN
+F 3 "" H 5800 7500 50  0001 C CNN
+	1    5800 7500
+	1    0    0    -1
+$EndComp
+Wire Wire Line
+	4750 7100 5000 7100
+Text Label 4750 7100 0    50   ~ 0
+IO5
+Wire Wire Line
+	5000 7300 4750 7300
+Wire Wire Line
+	5800 7200 6150 7200
+Connection ~ 5800 7200
+Text Label 6000 7200 0    50   ~ 0
+IO35
+Text Label 4750 7300 0    50   ~ 0
+GPIO0
 $EndSCHEMATC

Commit message: Changed the connectors from JST to a TE 1-1734595-2 connector.
This connector uses crimped on pins, but it may be easier to deal
with since it works with 28 gauge wire whereas the JST requires 30
gauge (though I ordered some 28AWG that should fit it).

This can always be reverted.

Signed-off-by: Aaron Williams <aaron.w2@gmail.com>
Parts:
- J2, J4: footprint aaron:BM12B-SRSS-TB -> aaron:TE_1_1734595_2_12Pos_1.0mm_Vert_SMD
Changed lines of the file:
@@
 F 0 "J4" H 5570 6367 50  0000 C CNN
 F 1 "Conn_01x12" H 5570 6276 50  0000 C CNN
-F 2 "aaron:BM12B-SRSS-TB" H 5650 5650 50  0001 C CNN
+F 2 "aaron:TE_1_1734595_2_12Pos_1.0mm_Vert_SMD" H 5650 5650 50  0001 C CNN
 F 3 "~" H 5650 5650 50  0001 C CNN
 	1    5650 5650
@@
 L Connector_Generic:Conn_01x12 J2
 U 1 1 5B9D440B
-P 3700 7100
-F 0 "J2" H 3620 7817 50  0000 C CNN
-F 1 "Conn_01x12" H 3620 7726 50  0000 C CNN
-F 2 "aaron:BM12B-SRSS-TB" H 3700 7100 50  0001 C CNN
-F 3 "~" H 3700 7100 50  0001 C CNN
-	1    3700 7100
-	-1   0    0    -1
+P 3700 7200
+F 0 "J2" H 3620 7917 50  0000 C CNN
+F 1 "Conn_01x12" H 3620 7826 50  0000 C CNN
+F 2 "aaron:TE_1_1734595_2_12Pos_1.0mm_Vert_SMD" H 3700 7200 50  0001 C CNN
+F 3 "~" H 3700 7200 50  0001 C CNN
+	1    3700 7200
+	-1   0    0    1
 $EndComp
 Wire Wire Line

Commit message: Finalized v1.4 design.
Added USB protection diodes.
Cleaned up routing some more.
Cleaned up the silk screening after getting connector models.

Signed-off-by: Aaron Williams <aaron.w2@gmail.com>
Parts:
- removed J7: Conn_01x02 DNS, Pin_Headers:Pin_Header_Straight_1x02_Pitch1.27mm, symbol Connector_Generic:Conn_01x02
- added D2: USBLC6-2SC6, TO_SOT_Packages_SMD:SOT-666, symbol dk_TVS-Diodes:USBLC6-2SC6
- added J7: Conn_01x03, Pin_Headers:Pin_Header_Straight_1x03_Pitch1.27mm, symbol Connector:Conn_01x03
- added Q4: BSS214NW, TO_SOT_Packages_SMD:SOT-323_SC-70, symbol Transistor_FET:BSS214NW
- added R11: 1m, Resistor_SMD:R_0603_1608Metric, symbol Device:R
- added R12: 22.1k, Resistor_SMD:R_0603_1608Metric, symbol device:R
- added R13: 47.5k, Resistor_SMD:R_0603_1608Metric, symbol device:R
- C1: value 10uF 10V -> 10uF; footprint Capacitors_SMD:C_0805 -> Capacitor_SMD:C_0805_2012Metric; MFR (none) -> Samsung; MPN (none) -> CL21B106KOQNNNE; Minimum Voltage (none) -> 10; SPN (none) -> 1276-2872-1-ND; SPR (none) -> Digikey; SPURL (none) -> -; Tolerance (none) -> 20%
- C10, C12, C13, C14, C2, C4, C6, C7, C9: value 10uF 10V -> 10uF; footprint Capacitors_SMD:C_0805 -> Capacitor_SMD:C_0805_2012Metric; MFR (none) -> Samsung; MPN (none) -> CL21B106KOQNNNE; SPN (none) -> 1276-2872-1-ND; SPR (none) -> Digikey; SPURL (none) -> -
- C11, C15, C16, C3, C8: value 1uF 10V -> 1uF; footprint Capacitors_SMD:C_0603 -> Capacitor_SMD:C_0603_1608Metric; MFR (none) -> Samsung; MPN (none) -> CL10B105KP8NNNC; SPN (none) -> 1276-1946-1-ND; SPR (none) -> Digikey; SPURL (none) -> -
- C5: value 0.1uF 10V -> 0.1uF; footprint Capacitors_SMD:C_0603 -> Capacitor_SMD:C_0603_1608Metric; MFR (none) -> Samsung; MPN (none) -> CL10B104KO8WPNC; SPN (none) -> 1276-6582-1-ND; SPR (none) -> Digikey; SPURL (none) -> -
- D1: MFR (none) -> Adafruit; MPN (none) -> 2686; SPN (none) -> 1528-1541-ND; SPR (none) -> Digikey; SPURL (none) -> -
- J1: MFR (none) -> Wuerth; MPN (none) -> 693072010801; SPN (none) -> 732-3820-1-ND; SPR (none) -> Digikey; SPURL (none) -> -
- J2, J4: footprint aaron:TE_1_1734595_2_12Pos_1.0mm_Vert_SMD -> Connectors_JST-BM12B-SURS-TF:BM12B-SRSS-TB; MFR (none) -> -; MPN (none) -> -; SPN (none) -> -; SPR (none) -> -; SPURL (none) -> -
- J3: MFR (none) -> Molex; MPN (none) -> 1050170001; SPN (none) -> WM1399CT-ND; SPR (none) -> Digikey; SPURL (none) -> -
- J5, J6, J8, U2: MFR (none) -> -; MPN (none) -> -; SPN (none) -> -; SPR (none) -> -; SPURL (none) -> -
- MIC1: MFR (none) -> SPH0645LM4H-B; SPN (none) -> 423-1405-1-ND; SPR (none) -> Digikey; SPURL (none) -> -
- Q1, Q2: MFR (none) -> Micro Commercial Co; SPN (none) -> MMBT2222ATPMSCT-ND; SPR (none) -> Digikey; SPURL (none) -> -
- Q3: MFR (none) -> ON Semiconductor; MPN (none) -> BSS138; SPN (none) -> BSS138CT-ND; SPR (none) -> Digikey; SPURL (none) -> -
- R1: footprint Resistors_SMD:R_0603 -> Resistor_SMD:R_0603_1608Metric; MFR (none) -> Vishay Dale; MPN (none) -> CRCW060310K0FKEC; SPN (none) -> 541-2979-1-ND; SPR (none) -> Digikey; SPURL (none) -> -; Tolerance (none) -> 5%
- R10: footprint Resistors_SMD:R_0603 -> Resistor_SMD:R_0603_1608Metric; MFR (none) -> Vishay Dale; MPN (none) -> CRCW0603100KJNEA; SPN (none) -> 541-100KGCT-ND; SPR (none) -> Digikey; SPURL (none) -> -
- R2: footprint Resistors_SMD:R_0603 -> Resistor_SMD:R_0603_1608Metric; MFR (none) -> Samsung; MPN (none) -> RC1608F471CS; SPN (none) -> 1276-4619-1-ND; SPR (none) -> Digikey; SPURL (none) -> -
- R3, R4, R5, R6, R7, R8, R9: footprint Resistors_SMD:R_0603 -> Resistor_SMD:R_0603_1608Metric; MFR (none) -> Vishay Dale; MPN (none) -> CRCW060310K0FKEC; SPN (none) -> 541-2979-1-ND; SPR (none) -> Digikey; SPURL (none) -> -
- RN1: footprint Resistors_SMD:R_Array_Convex_2x0603 -> Resistor_SMD:R_Array_Convex_2x0603; MFR (none) -> Panasonic; MPN (none) -> EXB-V4V103JV; SPN (none) -> Y2103CT-ND; SPR (none) -> Digikey; SPURL (none) -> -
- RN2: footprint Resistors_SMD:R_Array_Convex_4x0603 -> Resistor_SMD:R_Array_Convex_4x0603; MFR (none) -> Panasonic; MPN (none) -> EXB-V8V103JV; SPN (none) -> Y4103CT-ND; SPR (none) -> Digikey; SPURL (none) -> -
- SW1: footprint aaron:SW_SPST_KMR2 -> Buttons_Switches_SMD:SW_SPST_KMR2; MFR (none) -> C&K; MPN (none) -> KMR231NG LFS; SPN (none) -> CKN10246CT-ND; SPR (none) -> Digikey; SPURL (none) -> -
- U1: MFR (none) -> Torex Semiconductor; MPN (none) -> XCL220; SPN (none) -> 893-1279-1-ND; SPR (none) -> Digikey; SPURL (none) -> -
- U3: footprint Maxim:QFN-24-1EP_4x4mm_Pitch0.5mm -> Housings_DFN_QFN:QFN-24-1EP_4x4mm_Pitch0.5mm_rounded_corners; MFR (none) -> Silicon Image; MPN (none) -> CP2102N-A01-GQFN24; SPN (none) -> 336-4737-1-ND; SPR (none) -> Digikey; SPURL (none) -> -
- U4: MFR (none) -> Maxim; MPN (none) -> MAX14611ETD+T; SPN (none) -> MAX14611ETD+TCT-ND; SPR (none) -> Digikey; SPURL (none) -> -
Connections:
- net labels added: FET_1A, IO0, IO18_H, IO5_H
- net labels removed: GPIO0, IO25_H, IO26_H
- wire segments 247 -> 257
