File: led-controller-wrover32/led-controller-wrover32.sch (KiCad schematic (older format))
At the start: 51 parts, among them J1 Micro_SD_Card, J2 Conn_01x12, J3 USB_B_Micro, J4 Conn_01x12, J5 Conn_01x04 DNS, J6 Conn_01x02 DNS, J7 Conn_01x03, J8 Conn_01x05, Q1 MMBT2222A-TP, Q2 MMBT2222A-TP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

Commit message: Minor cleanup. - Removed overlapping fiducials (which aren't really needed) - Changed 3 pull-up resistors for IO21, IO22 and IO23 to use a   resistor network and moved further away from J8 - Fixed unconnected pull-up for IO15 (hopefully it was connected in 1.4) - Bumped to 1.4.2
Signed-off-by: Aaron Williams <aaron.w2@gmail.com>
Parts:
- removed R7, R8, R9: 10K, Resistor_SMD:R_0603_1608Metric, symbol Device:R
- added FID1, FID2, FID3: FIDUCIAL_1MM, Fiducials:Fiducial_0.5mm_Dia_1mm_Outer, symbol fiducial:FIDUCIAL_1MM
- added FID6: FIDUCIAL_1MM, Fiducials:Fiducial_1mm_Dia_2.54mm_Outer_CopperBottom, symbol fiducial:FIDUCIAL_1MM
- added RN3: R_Pack04, Resistor_SMD:R_Array_Concave_4x0603, symbol Device:R_Pack04
- D1: footprint LED_SMD:LED_SK6812MINI_PLCC4_3.5x3.5mm_P1.75mm -> Aaron:LED_SK6812MINI_PLCC4_3.5x3.5mm_P1.75mm
- D2: footprint TO_SOT_Packages_SMD:SOT-666 -> Package_TO_SOT_SMD:SOT-666; MFR (none) -> ST Microelectronics; SPN (none) -> 497-5026-1-ND; SPR (none) -> Digikey; SPURL (none) -> -
- J2, J4: MFR - -> JST; MPN - -> BM12B-SRSS-TF(LF)(SN); SPN - -> BM12B-SRSS-TF(LF)(SN)-ND; SPR - -> Digikey
- J3: footprint Connectors_USB:USB_Micro-B_Molex-105017-0001 -> Aaron:USB_Micro-B_Molex-105017-0001
- J7: value Conn_01x03 -> Conn_01x03 DNS
- Q1, Q2, Q3: footprint TO_SOT_Packages_SMD:SOT-23 -> Package_TO_SOT_SMD:SOT-23
- R12, R13: SPURL (none) -> -
- SW1: footprint Buttons_Switches_SMD:SW_SPST_KMR2 -> Aaron:SW_SPST_KMR2
- U1: MPN XCL220 -> XCL220B333FR-G
- U2: MFR - -> Espressif Systems; MPN - -> ESP32-WROVER-B (16MB); SPN - -> 356-ESP32-WROB(16MB); SPR - -> Mouser
- U3: footprint Housings_DFN_QFN:QFN-24-1EP_4x4mm_Pitch0.5mm_rounded_corners -> Aaron:QFN-24-1EP_4x4mm_Pitch0.5mm_rounded_corners
Connections:
- net labels added: IO27_5V
- wire segments 257 -> 237
