File: led-controller-wrover32/led-controller-wrover32.sch (KiCad schematic (older format))
At the start: 53 parts, among them J1 Micro_SD_Card, J2 Conn_01x12, J3 USB_B_Micro, J4 Conn_01x12, J5 Conn_01x04 DNS, J6 Conn_01x02 DNS, J7 Conn_01x03 DNS, J8 Conn_01x05, Q1 MMBT2222A-TP, Q2 MMBT2222A-TP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

Commit message: Fixed solder mask clearance.
Signed-off-by: Aaron Williams <aaron.w2@gmail.com>
Parts:
- removed FID6: FIDUCIAL_1MM, Fiducials:Fiducial_1mm_Dia_2.54mm_Outer_CopperBottom, symbol fiducial:FIDUCIAL_1MM
- removed R3, R4: 10K, Resistor_SMD:R_0603_1608Metric, symbol Device:R
- added RN4: R_Pack02, Resistor_SMD:R_Array_Convex_2x0603, symbol Device:R_Pack02
- RN3: footprint Resistor_SMD:R_Array_Concave_4x0603 -> Resistor_SMD:R_Array_Convex_4x0603
Connections:
- wire segments 237 -> 244
Changed lines of the file:
@@
 P 2450 1400
 F 0 "C2" H 2565 1446 50  0000 L CNN
-F 1 "10uF" H 2400 1150 50  0000 L CNN
+F 1 "10uF" H 2250 1500 50  0000 L CNN
 F 2 "Capacitor_SMD:C_0805_2012Metric" H 2488 1250 50  0001 C CNN
 F 3 "http://www.samsungsem.com/kr/support/product-search/mlcc/CL21B106KOQNNNE.jsp" H 2450 1400 50  0001 C CNN
@@
 P 2850 1400
 F 0 "C3" H 2965 1446 50  0000 L CNN
-F 1 "1uF" H 2550 1650 50  0000 L CNN
+F 1 "1uF" H 2900 1300 50  0000 L CNN
 F 2 "Capacitor_SMD:C_0603_1608Metric" H 2888 1250 50  0001 C CNN
 F 3 "http://www.samsungsem.com/kr/support/product-search/mlcc/CL10B105KP8NNNC.jsp" H 2850 1400 50  0001 C CNN
@@
 $EndComp
 $Comp
-L Device:R R4
-U 1 1 5B98BDF4
-P 9200 1550
-F 0 "R4" V 8993 1550 50  0000 C CNN
-F 1 "10K" V 9084 1550 50  0000 C CNN
-F 2 "Resistor_SMD:R_0603_1608Metric" V 9130 1550 50  0001 C CNN
-F 3 "http://www.vishay.com/docs/20035/dcrcwe3.pdf" H 9200 1550 50  0001 C CNN
-F 4 "Vishay Dale" H 0   0   50  0001 C CNN "MFR"
-F 5 "CRCW060310K0FKEC" H 0   0   50  0001 C CNN "MPN"
-F 6 "Digikey" H 0   0   50  0001 C CNN "SPR"
-F 7 "541-2979-1-ND" H 0   0   50  0001 C CNN "SPN"
-F 8 "-" H 0   0   50  0001 C CNN "SPURL"
-	1    9200 1550
-	0    1    1    0
-$EndComp
-$Comp
-L Device:R R3
-U 1 1 5B98BE71
-P 9200 950
-F 0 "R3" V 8993 950 50  0000 C CNN
-F 1 "10K" V 9084 950 50  0000 C CNN
-F 2 "Resistor_SMD:R_0603_1608Metric" V 9130 950 50  0001 C CNN
-F 3 "http://www.vishay.com/docs/20035/dcrcwe3.pdf" H 9200 950 50  0001 C CNN
-F 4 "Vishay Dale" H 0   0   50  0001 C CNN "MFR"
-F 5 "CRCW060310K0FKEC" H 0   0   50  0001 C CNN "MPN"
-F 6 "Digikey" H 0   0   50  0001 C CNN "SPR"
-F 7 "541-2979-1-ND" H 0   0   50  0001 C CNN "SPN"
-F 8 "-" H 0   0   50  0001 C CNN "SPURL"
-	1    9200 950
-	0    1    1    0
-$EndComp
-$Comp
 L MAX14611ETD_T:MAX14611ETD+T U4
 U 1 1 5B9A389B
@@
 Text Label 8650 950  0    50   ~ 0
 RTS
-Text Label 8650 1550 0    50   ~ 0
+Text Label 8650 1450 0    50   ~ 0
 DTR
 Text Label 10000 750  0    50   ~ 0
@@
 	4100 1100 4350 1100
 Wire Wire Line
-	9750 1150 9550 1350
-Wire Wire Line
-	9750 1350 9550 1150
+	9750 1150 9500 1400
+Wire Wire Line
+	9750 1350 9500 1100
 Wire Wire Line
 	9350 950  9450 950
 Wire Wire Line
-	9550 1150 9050 1150
-Wire Wire Line
-	9050 1150 9050 950
-Wire Wire Line
-	9350 1550 9450 1550
-Wire Wire Line
-	9050 1550 9050 1350
-Wire Wire Line
-	9050 1350 9550 1350
-Wire Wire Line
-	9050 1550 8650 1550
+	9050 1450 8650 1450
 Wire Wire Line
 	9750 750  10200 750
@@
 Connection ~ 7150 2750
 Connection ~ 6300 950
-Connection ~ 9050 950
-Connection ~ 9050 1550
 Connection ~ 10300 3450
 Connection ~ 9950 3350
@@
 	1    0    0    -1
 $EndComp
-$Comp
-L fiducial:FIDUCIAL_1MM FID6
-U 1 1 5BBF9E61
-P 9650 6500
-F 0 "FID6" H 9753 6606 60  0000 L CNN
-F 1 "FIDUCIAL_1MM" H 9753 6500 60  0000 L CNN
-F 2 "Fiducials:Fiducial_1mm_Dia_2.54mm_Outer_CopperBottom" H 9753 6394 60  0000 L CNN
-F 3 "" H 9650 6500 60  0000 C CNN
-	1    9650 6500
-	1    0    0    -1
-$EndComp
 Text Label 9500 2550 2    50   ~ 0
 IO27_5V
@@
 	7900 950  7900 1450
 Wire Wire Line
-	7900 950  9050 950
-Wire Wire Line
-	8650 1850 8650 1550
+	8650 1850 8650 1450
 Wire Wire Line
 	7750 1850 8650 1850
@@
 F 0 "RN3" H 8120 5446 50  0000 R CNN
 F 1 "R_Pack04" H 8120 5355 50  0000 R CNN
-F 2 "Resistor_SMD:R_Array_Concave_4x0603" V 8675 5400 50  0001 C CNN
+F 2 "Resistor_SMD:R_Array_Convex_4x0603" V 8675 5400 50  0001 C CNN
 F 3 "~" H 8400 5400 50  0001 C CNN
 	1    8400 5400
@@
 	8500 5200 8400 5200
 Connection ~ 8500 5200
+$Comp
+L Device:R_Pack02 RN4
+U 1 1 5BC02AB8
+P 8850 1300
+F 0 "RN4" V 8533 1300 50  0000 C CNN
+F 1 "R_Pack02" V 8624 1300 50  0000 C CNN
+F 2 "Resistor_SMD:R_Array_Convex_2x0603" V 9025 1300 50  0001 C CNN
+F 3 "https://industrial.panasonic.com/cdbs/www-data/pdf/AOC0000/AOC0000C14.pdf" H 8850 1300 50  0001 C CNN
+F 4 "Panasonic" H 6950 -3750 50  0001 C CNN "MFR"
+F 5 "EXB-V4V103JV" H 6950 -3750 50  0001 C CNN "MPN"
+F 6 "Digikey" H 6950 -3750 50  0001 C CNN "SPR"
+F 7 "Y2103CT-ND" H 6950 -3750 50  0001 C CNN "SPN"
+F 8 "-" H 6950 -3750 50  0001 C CNN "SPURL"
+	1    8850 1300
+	0    -1   1    0
+$EndComp
+Wire Wire Line
+	8650 1200 8650 950
+Wire Wire Line
+	9200 1100 9050 950
+Wire Wire Line
+	9050 1200 9350 1200
+Wire Wire Line
+	9350 1200 9350 950
+Wire Wire Line
+	9500 1100 9200 1100
+Connection ~ 8650 950
+Wire Wire Line
+	8650 950  9050 950
+Wire Wire Line
+	7900 950  8650 950
+Wire Wire Line
+	9050 1300 9050 1400
+Connection ~ 9050 1400
+Wire Wire Line
+	9050 1400 9050 1450
+Wire Wire Line
+	9050 1400 9500 1400
+Wire Wire Line
+	8550 1550 8550 1300
+Wire Wire Line
+	8550 1300 8650 1300
+Wire Wire Line
+	8550 1550 9450 1550
 $EndSCHEMATC

Commit message: - Cleaned up the schematic - Made J5 USB D+ and D- go through protection diodes
Signed-off-by: Aaron Williams <aaron.w2@gmail.com>
Parts:
- D1: value SK6812MINI -> WS1812B 3535
- RN1, RN4: value R_Pack02 -> 10K
- RN2: value R_Pack04 -> 10K
- U1: value XCL21X -> XCL220
Connections:
- net labels added: D+, D-
- wire segments 244 -> 231
- no-connect marks 0 -> 20
Other:
- note added: "* Technically no more than 500ma can be drawn from USB alone"
- note added: "3.3V to 5V level shifter"
- note added: "3V to 5V level shifter and WS1812B 3535\nNote output goes to J2 pin 4"
- note added: "5V to 3.3V Buck Regulator\n1A maximum output"
- note added: "AUX Power Input/Output connectors"
- note added: "Aux I/O connector for I2C + interrupts\nDuplicate I/Os from J4"
- note added: "Espressif ESP32 Wrover module and SD connector"
- note added: "I2S microphone\nNote that IO0, IO19\nand IO35 are shared\nwith J4. Microphone\nwired for left channel."
- note added: "J7 pin 3 can be used for PWM.\nNote that Wrover32 IO26\ncan do analog output."
- note added: "Main I/O connectors"
- note added: "Place near\nUSB conn"
- note added: "Reset button"
- note added: "Reset/Programming circuit copied from Adafruit"
- note added: "USB to Serial Programmer"
- note added: "Use either J3 or J5 for USB signals, not both"
- note removed: "Place near ESP32"
- moved on the sheet: C10, C11, C12, C13, C14, C15, C16, C2, C3, C5, C7, C8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

Commit message: Fixed (hopefully) the ws1812b 3535 footprint.
Signed-off-by: Aaron Williams <aaron.w2@gmail.com>
Parts:
- J7: symbol Connector:Conn_01x03 -> led-controller-wrover32-rescue:Conn_01x03-Connector
- J8: symbol Connector:Conn_01x05 -> led-controller-wrover32-rescue:Conn_01x05-Connector
- R12, R13: symbol device:R -> led-controller-wrover32-rescue:R-device
- SW1: footprint Aaron:SW_SPST_KMR2 -> Button_Switch_SMD:SW_SPST_KMR2
Changed lines of the file:
@@
 Sheet 1 1
 Title "Wrover32 LED Controller"
-Date ""
-Rev "1.4.4"
+Date "2018-11-05"
+Rev "1.4.5"
 Comp ""
 Comment1 "Copyright © 2018 by Aaron Williams"
@@
 F 0 "SW1" V 6340 5559 42  0000 R CNN
 F 1 "KMR2" V 6261 5559 42  0000 R CNN
-F 2 "Aaron:SW_SPST_KMR2" H 6300 5700 50  0001 C CNN
+F 2 "Button_Switch_SMD:SW_SPST_KMR2" H 6300 5700 50  0001 C CNN
 F 3 "https://www.ckswitches.com/media/1479/kmr2.pdf" H 6300 5700 50  0001 C CNN
 F 4 "C&K" H 1800 4100 50  0001 C CNN "MFR"
@@
 $EndComp
 $Comp
-L Connector:Conn_01x05 J8
+L led-controller-wrover32-rescue:Conn_01x05-Connector J8
 U 1 1 5BAE7406
 P 8800 6050
@@
 $EndComp
 $Comp
-L Connector:Conn_01x03 J7
+L led-controller-wrover32-rescue:Conn_01x03-Connector J7
 U 1 1 5BB02006
 P 700 2400
@@
 $EndComp
 $Comp
-L device:R R12
+L led-controller-wrover32-rescue:R-device R12
 U 1 1 5BB18E30
 P 5650 1000
@@
 $EndComp
 $Comp
-L device:R R13
+L led-controller-wrover32-rescue:R-device R13
 U 1 1 5BB18EB8
 P 5650 1300
@@
 	2150 1400 2150 1250
 Wire Wire Line
-	2700 1700 2300 1700
-Wire Wire Line
 	2300 1400 2700 1400
 Wire Wire Line
@@
 Connection ~ 850  1050
 Connection ~ 1550 1800
-Connection ~ 2700 1700
 Connection ~ 2300 1400
-Connection ~ 2700 1400
 Connection ~ 7150 2750
 Connection ~ 10100 3750
@@
 	500  6500 2800 6500
 Wire Notes Line
-	2800 6500 2800 8000
-Wire Notes Line
 	10400 3300 7150 3300
 Wire Notes Line
@@
 Connection ~ 10150 2450
 Connection ~ 10150 3100
+Wire Notes Line
+	2800 6500 2800 8000
+Wire Wire Line
+	2700 1700 2300 1700
+Connection ~ 2700 1400
+Connection ~ 2700 1700
 $EndSCHEMATC

Commit message: This fixes a number of issues: - IO2 is now set according to the DTR and RTS signals.  This is required for   booting over the serial port. - Some more footprints were found to be using the old Kicad 4 footprints and   have been changed to KiCad 5. - One more fidicial has been added - More capacitors have been added. 	- 10uF for Wrover32 increased to 22uF 	- Some 1uF were changed to 0.1uF
Signed-off-by: Aaron Williams <aaron.w2@gmail.com>
Parts:
- removed Q1: MMBT2222A-TP, Package_TO_SOT_SMD:SOT-23, symbol dk_Transistors-Bipolar-BJT-Single:MMBT2222A-TP
- removed RN4: 10K, Resistor_SMD:R_Array_Convex_2x0603, symbol Device:R_Pack02
- added C17: 0.1uF, Capacitor_SMD:C_0603_1608Metric, symbol Device:C
- added C18: 10uF, Capacitor_SMD:C_0805_2012Metric, symbol Device:C
- added FID4: FIDUCIAL_1MM, Fiducial:Fiducial_0.5mm_Dia_1mm_Outer, symbol fiducial:FIDUCIAL_1MM
- added Q1: MMDT5551, Package_TO_SOT_SMD:SOT-363_SC-70-6, symbol Transistor_BJT:MMDT5551
- added RN4: 10K, Resistor_SMD:R_Array_Convex_4x0603, symbol Device:R_Pack04
- C12: value 10uF -> 22uF; MPN CL21B106KOQNNNE -> CL21A226KPCLRNC; SPN 1276-2872-1-ND -> 1276-6786-1-ND; SPURL - -> https://www.digikey.com/product-detail/en/samsung-electro-m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
- C16, C8: value 1uF -> 0.1uF; MFR Samsung -> AVX; MPN CL10B105KP8NNNC -> 06035C104K4Z4A; SPN 1276-1946-1-ND -> 478-10679-1-ND; SPURL - -> https://www.digikey.com/product-detail/en/avx-corporation/0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
- FID1, FID2, FID3: footprint Fiducials:Fiducial_0.5mm_Dia_1mm_Outer -> Fiducial:Fiducial_0.5mm_Dia_1mm_Outer
- J1: footprint Connectors:microSD_Card_Receptacle_Wuerth_693072010801 -> Connector_Card:microSD_HC_Wuerth_693072010801
- J5: footprint Pin_Headers:Pin_Header_Straight_1x04_Pitch2.54mm -> Connector_PinHeader_2.54mm:PinHeader_1x04_P2.54mm_Vertical
- J6: footprint Pin_Headers:Pin_Header_Straight_1x02_Pitch1.27mm -> Connector_PinHeader_1.27mm:PinHeader_1x02_P1.27mm_Vertical
- J7: footprint Pin_Headers:Pin_Header_Straight_1x03_Pitch1.27mm -> Connector_PinHeader_1.27mm:PinHeader_1x03_P1.27mm_Vertical; symbol led-controller-wrover32-rescue:Conn_01x03-Connector -> led-controller-wrover32-rescue:Conn_01x03-Connector-led-controller-wrover32-rescue
- J8: footprint Pin_Headers:Pin_Header_Straight_1x05_Pitch1.27mm -> Connector_PinHeader_1.27mm:PinHeader_1x05_P1.27mm_Vertical; symbol led-controller-wrover32-rescue:Conn_01x05-Connector -> led-controller-wrover32-rescue:Conn_01x05-Connector-led-controller-wrover32-rescue
- R12, R13: symbol led-controller-wrover32-rescue:R-device -> led-controller-wrover32-rescue:R-device-led-controller-wrover32-rescue
- SW1: footprint Button_Switch_SMD:SW_SPST_KMR2 -> Aaron:SW_SPST_KMR2
Connections:
- wire segments 231 -> 249
- no-connect marks 20 -> 22
Other:
- note added: "Reset/Programming circuit"
- note removed: "Reset/Programming circuit copied from Adafruit"

Commit message: Updated README.md and added BOM.  Note that there were no changes to the board layout.
Signed-off-by: Aaron Williams <aaron.w2@gmail.com>
Parts:
- C16, C17, C8: MFR AVX -> Samsung; MPN 06035C104K4Z4A -> CL10B104KO8WPNC; SPN 478-10679-1-ND -> 1276-6582-1-ND
- FID1, FID2, FID3, FID4, RN3: MFR (none) -> -; MPN (none) -> -; SPN (none) -> -; SPR (none) -> -; SPURL (none) -> -
- J1: footprint Connector_Card:microSD_HC_Wuerth_693072010801 -> Aaron:microSD_HC_Wuerth_693072010801
- J7: symbol led-controller-wrover32-rescue:Conn_01x03-Connector-led-controller-wrover32-rescue -> led-controller-wrover32-rescue:Conn_01x03-Connector-led-controller-wrover32-rescue-led-controller-wrover32-rescue
- J8: symbol led-controller-wrover32-rescue:Conn_01x05-Connector-led-controller-wrover32-rescue -> led-controller-wrover32-rescue:Conn_01x05-Connector-led-controller-wrover32-rescue-led-controller-wrover32-rescue
- Q1: MFR (none) -> Diodes, Inc.; MPN (none) -> MMDT5551-7-F; SPN (none) -> MMDT5551-FDICT-ND; SPR (none) -> Digikey; SPURL (none) -> -
- R12, R13: symbol led-controller-wrover32-rescue:R-device-led-controller-wrover32-rescue -> led-controller-wrover32-rescue:R-device-led-controller-wrover32-rescue-led-controller-wrover32-rescue

Commit message: Fixed value for RN3 and fidicial references and added rescue files.
Signed-off-by: Aaron Williams <aaron.w2@gmail.com>
Parts:
- RN3: value R_Pack04 -> 10K; MFR - -> Panasonic; MPN - -> EXB-V8V103JV; SPN - -> Y4103CT-ND; SPR - -> Digikey
Changed lines of the file:
@@
 P 8000 5600
 F 0 "RN3" H 8350 5700 50 0000 R CNN
-F 1 "R_Pack04" H 8550 5600 50 0000 R CNN
+F 1 "10K" H 8350 5600 50 0000 R CNN
 F 2 "Resistor_SMD:R_Array_Convex_4x0603" V 8275 5600 50 0001 C CNN
-F 3 "~" H 8000 5600 50 0001 C CNN
-F 4 "-" H 0 0 50 0001 C CNN "MFR"
-F 5 "-" H 0 0 50 0001 C CNN "MPN"
-F 6 "-" H 0 0 50 0001 C CNN "SPR"
-F 7 "-" H 0 0 50 0001 C CNN "SPN"
+F 3 "https://industrial.panasonic.com/cdbs/www-data/pdf/AOC0000/AOC0000C14.pdf" H 8000 5600 50 0001 C CNN
+F 4 "Panasonic" H 0 0 50 0001 C CNN "MFR"
+F 5 "EXB-V8V103JV" H 0 0 50 0001 C CNN "MPN"
+F 6 "Digikey" H 0 0 50 0001 C CNN "SPR"
+F 7 "Y4103CT-ND" H 0 0 50 0001 C CNN "SPN"
 F 8 "-" H 0 0 50 0001 C CNN "SPURL"
 	1    8000 5600
