File: led-controller-wrover32/12v-booster.sch (KiCad schematic (older format))
At the start: 16 parts, among them J101 Conn_01x02 DNS, U101 TPS55340-Q1

Commit message: Minor changes.
Signed-off-by: Aaron Williams <aaron.w2@gmail.com>
Parts:
- D101: value D_Schottky -> Shottkey SS24FL
- J101: value Conn_01x02 DNS -> B2B-PH-K-S(LF)(SN) DNS
