File: led-controller-wrover32/12v-booster.sch (KiCad schematic (older format))
At the start: 16 parts, among them J101 Conn_01x02, U101 TPS55340-Q1

Commit message: Minor changes
- Tweaked some of the component values in the 12V supply as per TI.
- Removed unnecessary protection diode, the USB one is enough.
- Changed UART to CS2104 which eliminates two resistors and is
  slightly cheaper
- Updated PCB to reflect changes.

Signed-off-by: Aaron Williams <aaron.w2@gmail.com>
Parts:
- C101: value 6.8uF -> 22uF; DESC (none) -> CAP CER 22UF 16V X5R 0603; MFR TDK -> Samsung Electro-Mechanics; MPN C1608X5R1E685K080AC -> CL10A226MO7JZNC; SPN 445-14145-1-ND -> 1276-7076-1-ND; SPURL - -> https://www.digikey.com/products/en/capacitors/ceramic-capa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
- C102, C108: DESC (none) -> CAP CER 0.1UF 50V X7R 0603
- C103: value 22uF -> 47uF; DESC (none) -> CAP CER 47UF 16V X5R 1210; MPN CL32B226MOJNNNE -> CL32A476KOJNNNE; SPN 1276-3395-1-ND -> 1276-3376-1-ND; SPURL - -> https://www.digikey.com/product-detail/en/samsung-electro-m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
- C104: DESC (none) -> CAP CER 1UF 10V X7R 0603
- C105: DESC (none) -> CAP CER 0.022UF 50V X7R 0603
- C106: DESC (none) -> CAP CER 820PF 50V C0G/NPO 0603
- C107: DESC (none) -> CAP CER 0.47UF 50V X5R 0603
- D101: DESC (none) -> DIODE SCHOTTKY 40V 2A SOD123F
- J101: DESC (none) -> CONN HEADER VERT 2POS 2MM
- L101: DESC (none) -> FIXED IND 3.3UH 2.7A 61 MOHM SMD
- R101: DESC (none) -> RES SMD 86.6K OHM 1% 1/10W 0603
- R102: value 18.2K -> 18.7K; DESC (none) -> RES SMD 18.7K OHM 1% 1/10W 0603; MFR Vishay Dale -> Yageo; MPN CRCW060318K2FKEA -> RC0603FR-0718K7L; SPN 541-18.2KHCT-ND -> 311-18.7KHRCT-ND; SPURL - -> https://www.digikey.com/product-detail/en/yageo/RC0603FR-07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
- R103: value 1.69K -> 1.62K; DESC (none) -> RES SMD 1.62K OHM 1% 1/10W 0603; MFR Vishay -> Yageo; MPN CRCW06031K69FKEA -> RC0603FR-071K62L; SPN 541-1.69KHCT-ND -> 311-1.62KHRCT-ND; SPURL - -> https://www.digikey.com/product-detail/en/yageo/RC0603FR-07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
- R104: DESC (none) -> RES SMD 10K OHM 1% 1/10W 0603
- U101: DESC (none) -> IC REG BOOST ADJ 5.25A 16WQFN; MFR TI -> Texas Instruments
Changed lines of the file:
@@
 F 2 "Aaron:QFN-16-1EP_3x3mm_P0.5mm_EP2.7x2.7mm_ThermalVias" H 4950 3000 50  0001 C CNN
 F 3 "http://www.ti.com/lit/ds/symlink/tps55340-q1.pdf" H 4950 3000 50  0001 C CNN
-F 4 "TI" H 0   0   50  0001 C CNN "MFR"
+F 4 "Texas Instruments" H 0   0   50  0001 C CNN "MFR"
 F 5 "TPS55340RTER" H 0   0   50  0001 C CNN "MPN"
 F 6 "Digikey" H 0   0   50  0001 C CNN "SPR"
 F 7 "296-37677-1-ND" H 0   0   50  0001 C CNN "SPN"
 F 8 "-" H 0   0   50  0001 C CNN "SPURL"
+F 9 "IC REG BOOST ADJ 5.25A 16WQFN" H 0   0   50  0001 C CNN "DESC"
 	1    4950 3000
 	1    0    0    -1
@@
 F 7 "541-2567-1-ND" H 0   0   50  0001 C CNN "SPN"
 F 8 "-" H 0   0   50  0001 C CNN "SPURL"
+F 9 "FIXED IND 3.3UH 2.7A 61 MOHM SMD" H 0   0   50  0001 C CNN "DESC"
 	1    4950 1900
 	0    -1   -1   0
@@
 F 7 "SS24FLCT-ND" H 0   0   50  0001 C CNN "SPN"
 F 8 "-" H 0   0   50  0001 C CNN "SPURL"
+F 9 "DIODE SCHOTTKY 40V 2A SOD123F" H 0   0   50  0001 C CNN "DESC"
 	1    6300 2450
 	-1   0    0    1
@@
 P 2800 2750
 F 0 "C101" H 2915 2796 50  0000 L CNN
-F 1 "6.8uF" H 2915 2705 50  0000 L CNN
+F 1 "22uF" H 2915 2705 50  0000 L CNN
 F 2 "Capacitor_SMD:C_0603_1608Metric" H 2838 2600 50  0001 C CNN
-F 3 "https://product.tdk.com/info/en/catalog/datasheets/mlcc_commercial_general_en.pdf" H 2800 2750 50  0001 C CNN
-F 4 "TDK" H 0   0   50  0001 C CNN "MFR"
-F 5 "C1608X5R1E685K080AC" H 0   0   50  0001 C CNN "MPN"
-F 6 "Digikey" H 0   0   50  0001 C CNN "SPR"
-F 7 "445-14145-1-ND" H 0   0   50  0001 C CNN "SPN"
-F 8 "-" H 0   0   50  0001 C CNN "SPURL"
+F 3 "http://www.samsungsem.com/kr/support/product-search/mlcc/CL10A226MO7JZNC.jsp" H 2800 2750 50  0001 C CNN
+F 4 "Samsung Electro-Mechanics" H 0   0   50  0001 C CNN "MFR"
+F 5 "CL10A226MO7JZNC" H 0   0   50  0001 C CNN "MPN"
+F 6 "Digikey" H 0   0   50  0001 C CNN "SPR"
+F 7 "1276-7076-1-ND" H 0   0   50  0001 C CNN "SPN"
+F 8 "https://www.digikey.com/products/en/capacitors/ceramic-capacitors/60?k=&pkeyword=&sv=0&pv2049=u22%C2%B5F&sf=1&FV=7%7C2%2C14%7C108742%2C17%7C422407%2C17%7C422415%2C1989%7C0%2C-8%7C60%2C16%7C39246%2C69%7C409416&quantity=&ColumnSort=0&page=1&stock=1&nstock=1&pageSize=500" H 0   0   50  0001 C CNN "SPURL"
+F 9 "CAP CER 22UF 16V X5R 0603" H 0   0   50  0001 C CNN "DESC"
 	1    2800 2750
-	1    0    0    -1
-$EndComp
-$Comp
-L Device:C C102
-U 1 1 5BAB11A4
-P 3200 2750
-F 0 "C102" H 3315 2796 50  0000 L CNN
-F 1 "0.1uF" H 3315 2705 50  0000 L CNN
-F 2 "Capacitor_SMD:C_0603_1608Metric" H 3238 2600 50  0001 C CNN
-F 3 "https://psearch.en.murata.com/capacitor/product/GCM188R71H104KA57%23.pdf" H 3200 2750 50  0001 C CNN
-F 4 "Murata Electronics" H 0   0   50  0001 C CNN "MFR"
-F 5 "GCM188R71H104KA57D" H 0   0   50  0001 C CNN "MPN"
-F 6 "Digikey" H 0   0   50  0001 C CNN "SPR"
-F 7 "490-4779-1-ND" H 0   0   50  0001 C CNN "SPN"
-F 8 "-" H 0   0   50  0001 C CNN "SPURL"
-	1    3200 2750
 	1    0    0    -1
 $EndComp
@@
 P 3700 2950
 F 0 "R102" H 3770 2996 50  0000 L CNN
-F 1 "18.2K" H 3770 2905 50  0000 L CNN
+F 1 "18.7K" H 3770 2905 50  0000 L CNN
 F 2 "Resistor_SMD:R_0603_1608Metric" V 3630 2950 50  0001 C CNN
-F 3 "~" H 3700 2950 50  0001 C CNN
-F 4 "Vishay Dale" H 0   0   50  0001 C CNN "MFR"
-F 5 "CRCW060318K2FKEA" H 0   0   50  0001 C CNN "MPN"
-F 6 "Digikey" H 0   0   50  0001 C CNN "SPR"
-F 7 "541-18.2KHCT-ND" H 0   0   50  0001 C CNN "SPN"
-F 8 "-" H 0   0   50  0001 C CNN "SPURL"
+F 3 "https://www.yageo.com/upload/media/product/productsearch/datasheet/rchip/PYu-RC_Group_51_RoHS_L_10.pdf" H 3700 2950 50  0001 C CNN
+F 4 "Yageo" H 0   0   50  0001 C CNN "MFR"
+F 5 "RC0603FR-0718K7L" H 0   0   50  0001 C CNN "MPN"
+F 6 "Digikey" H 0   0   50  0001 C CNN "SPR"
+F 7 "311-18.7KHRCT-ND" H 0   0   50  0001 C CNN "SPN"
+F 8 "https://www.digikey.com/product-detail/en/yageo/RC0603FR-0718K7L/311-18.7KHRCT-ND/729940" H 0   0   50  0001 C CNN "SPURL"
+F 9 "RES SMD 18.7K OHM 1% 1/10W 0603" H 0   0   50  0001 C CNN "DESC"
 	1    3700 2950
 	1    0    0    -1
@@
 F 7 "311-4010-1-ND" H 0   0   50  0001 C CNN "SPN"
 F 8 "https://www.digikey.com/product-detail/en/yageo/CC0603JRX7R9BB223/311-4010-1-ND/8025099" H 0   0   50  0001 C CNN "SPURL"
+F 9 "CAP CER 0.022UF 50V X7R 0603" H 0   0   50  0001 C CNN "DESC"
 	1    3950 3550
 	1    0    0    -1
@@
 F 7 "311-1775-1-ND" H 0   0   50  0001 C CNN "SPN"
 F 8 "https://www.digikey.com/products/en?keywords=311-1775-1-ND" H 0   0   50  0001 C CNN "SPURL"
+F 9 "CAP CER 820PF 50V C0G/NPO 0603" H 0   0   50  0001 C CNN "DESC"
 	1    5850 3600
 	1    0    0    -1
-$EndComp
-$Comp
-L Device:R R103
-U 1 1 5BAB141D
-P 6400 3300
-F 0 "R103" V 6193 3300 50  0000 C CNN
-F 1 "1.69K" V 6284 3300 50  0000 C CNN
-F 2 "Resistor_SMD:R_0603_1608Metric" V 6330 3300 50  0001 C CNN
-F 3 "http://www.vishay.com/docs/20035/dcrcwe3.pdf" H 6400 3300 50  0001 C CNN
-F 4 "Vishay" H 250 300 50  0001 C CNN "MFR"
-F 5 "CRCW06031K69FKEA" H 250 300 50  0001 C CNN "MPN"
-F 6 "Digikey" H 250 300 50  0001 C CNN "SPR"
-F 7 "541-1.69KHCT-ND" H 250 300 50  0001 C CNN "SPN"
-F 8 "-" H 250 300 50  0001 C CNN "SPURL"
-	1    6400 3300
-	-1   0    0    1
 $EndComp
 $Comp
@@
 F 7 "490-11994-1-ND" H 0   0   50  0001 C CNN "SPN"
 F 8 "-" H 0   0   50  0001 C CNN "SPURL"
+F 9 "CAP CER 0.47UF 50V X5R 0603" H 0   0   50  0001 C CNN "DESC"
 	1    6400 3600
 	1    0    0    -1
@@
 F 7 "541-2979-1-ND" H 0   0   50  0001 C CNN "SPN"
 F 8 "-" H 0   0   50  0001 C CNN "SPURL"
+F 9 "RES SMD 10K OHM 1% 1/10W 0603" H 0   0   50  0001 C CNN "DESC"
 	1    7100 3250
 	1    0    0    -1
@@
 F 7 "541-86.6KHCT-ND" H 0   0   50  0001 C CNN "SPN"
 F 8 "-" H 0   0   50  0001 C CNN "SPURL"
+F 9 "RES SMD 86.6K OHM 1% 1/10W 0603" H 0   0   50  0001 C CNN "DESC"
 	1    7100 2600
 	1    0    0    -1
@@
 P 7550 2850
 F 0 "C103" H 7665 2896 50  0000 L CNN
-F 1 "22uF" H 7665 2805 50  0000 L CNN
+F 1 "47uF" H 7665 2805 50  0000 L CNN
 F 2 "Capacitor_SMD:C_1210_3225Metric" H 7588 2700 50  0001 C CNN
-F 3 "http://www.samsungsem.com/kr/support/product-search/mlcc/CL32B226MOJNNNE.jsp" H 7550 2850 50  0001 C CNN
+F 3 "http://www.samsungsem.com/kr/support/product-search/mlcc/CL32A476KOJNNNE.jsp" H 7550 2850 50  0001 C CNN
 F 4 "Samsung" H 0   0   50  0001 C CNN "MFR"
-F 5 "CL32B226MOJNNNE" H 0   0   50  0001 C CNN "MPN"
-F 6 "Digikey" H 0   0   50  0001 C CNN "SPR"
-F 7 "1276-3395-1-ND" H 0   0   50  0001 C CNN "SPN"
-F 8 "-" H 0   0   50  0001 C CNN "SPURL"
+F 5 "CL32A476KOJNNNE" H 0   0   50  0001 C CNN "MPN"
+F 6 "Digikey" H 0   0   50  0001 C CNN "SPR"
+F 7 "1276-3376-1-ND" H 0   0   50  0001 C CNN "SPN"
+F 8 "https://www.digikey.com/product-detail/en/samsung-electro-mechanics/CL32A476KOJNNNE/1276-3376-1-ND/3891462" H 0   0   50  0001 C CNN "SPURL"
+F 9 "CAP CER 47UF 16V X5R 1210" H 0   0   50  0001 C CNN "DESC"
 	1    7550 2850
 	1    0    0    -1
@@
 F 7 "1276-1946-1-ND" H 0   0   50  0001 C CNN "SPN"
 F 8 "-" H 0   0   50  0001 C CNN "SPURL"
+F 9 "CAP CER 1UF 10V X7R 0603" H 0   0   50  0001 C CNN "DESC"
 	1    8000 2850
 	1    0    0    -1
@@
 F 7 "Digikey" H 9100 2550 50  0001 C CNN "SPR"
 F 8 "https://www.digikey.com/product-detail/en/jst-sales-america-inc/B2B-PH-K-S-LF-SN/455-1704-ND/926611" H 9100 2550 50  0001 C CNN "SPURL"
+F 9 "CONN HEADER VERT 2POS 2MM" H 0   0   50  0001 C CNN "DESC"
 	1    9100 2550
 	1    0    0    1
@@
 F 7 "Digikey" H 8500 2850 50  0001 C CNN "SPR"
 F 8 "https://www.digikey.com/product-detail/en/murata-electronics/GCM188R71H104KA57D/490-4779-1-ND/1641698" H 8500 2850 50  0001 C CNN "SPURL"
+F 9 "CAP CER 0.1UF 50V X7R 0603" H 0   0   50  0001 C CNN "DESC"
 	1    8500 2850
 	1    0    0    -1
@@
 F 3 "~" H 8500 2450 50  0001 C CNN
 	1    8500 2450
+	1    0    0    -1
+$EndComp
+$Comp
+L Device:C C102
+U 1 1 5BAB11A4
+P 3200 2750
+F 0 "C102" H 3315 2796 50  0000 L CNN
+F 1 "0.1uF" H 3315 2705 50  0000 L CNN
+F 2 "Capacitor_SMD:C_0603_1608Metric" H 3238 2600 50  0001 C CNN
+F 3 "https://psearch.en.murata.com/capacitor/product/GCM188R71H104KA57%23.pdf" H 3200 2750 50  0001 C CNN
+F 4 "Murata Electronics" H 0   0   50  0001 C CNN "MFR"
+F 5 "GCM188R71H104KA57D" H 0   0   50  0001 C CNN "MPN"
+F 6 "Digikey" H 0   0   50  0001 C CNN "SPR"
+F 7 "490-4779-1-ND" H 0   0   50  0001 C CNN "SPN"
+F 8 "-" H 0   0   50  0001 C CNN "SPURL"
+F 9 "CAP CER 0.1UF 50V X7R 0603" H 0   0   50  0001 C CNN "DESC"
+	1    3200 2750
 	1    0    0    -1
 $EndComp
@@
 Connection ~ 8900 3750
 NoConn ~ 5500 3900
+$Comp
+L Device:R R103
+U 1 1 5BAB141D
+P 6400 3300
+F 0 "R103" V 6193 3300 50  0000 C CNN
+F 1 "1.62K" V 6284 3300 50  0000 C CNN
+F 2 "Resistor_SMD:R_0603_1608Metric" V 6330 3300 50  0001 C CNN
+F 3 "https://www.yageo.com/upload/media/product/productsearch/datasheet/rchip/PYu-RC_Group_51_RoHS_L_10.pdf" H 6400 3300 50  0001 C CNN
+F 4 "Yageo" H 250 300 50  0001 C CNN "MFR"
+F 5 "RC0603FR-071K62L" H 250 300 50  0001 C CNN "MPN"
+F 6 "Digikey" H 250 300 50  0001 C CNN "SPR"
+F 7 "311-1.62KHRCT-ND" H 250 300 50  0001 C CNN "SPN"
+F 8 "https://www.digikey.com/product-detail/en/yageo/RC0603FR-071K62L/311-1.62KHRCT-ND/729816" H 250 300 50  0001 C CNN "SPURL"
+F 9 "RES SMD 1.62K OHM 1% 1/10W 0603" H 0   0   50  0001 C CNN "DESC"
+	1    6400 3300
+	-1   0    0    1
+$EndComp
 $EndSCHEMATC

Commit message: Multiple changes from v3.7
1. Fixed microphone so it uses the left channel
2. Reduced the number of unique components, i.e. replacing a couple of
   resistor networks with already used resistors
3. Removed unneeded resistor in programming circuit
4. Moved speaker chip to the other side to be closer to the connector
5. Cleaned up some of the traces and removed some inner-layer traces.
6. Moved reset switch to the edge to make access easier.
7. Added big via to line up with daughter card.
8. Replaced BSS138 transistor array with two BSS138 transistors to reduce
   the unique component count and reduce cost.

Signed-off-by: Aaron Williams <aaron.w2@gmail.com>
Parts:
- C102: SPURL - -> https://www.digikey.com/product-detail/en/murata-electronic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
- C104: SPURL - -> https://www.digikey.com/products/en?keywords=1276-1946-1-ND
- C107: SPURL - -> https://www.digikey.com/products/en?keywords=490-11994-1-ND
- D101: SPURL - -> https://www.digikey.com/products/en?keywords=SS24FLCT-ND
- L101: SPURL - -> https://www.digikey.com/products/en?keywords=541-2567-1-ND
- R101: SPURL - -> https://www.digikey.com/products/en?keywords=541-86.6KHCT-ND
- R104: SPURL - -> https://www.digikey.com/products/en?keywords=541-2979-1-ND
- U101: SPURL - -> https://www.digikey.com/products/en?keywords=296-37677-1-ND
Changed lines of the file:
@@
 F 6 "Digikey" H 0   0   50  0001 C CNN "SPR"
 F 7 "296-37677-1-ND" H 0   0   50  0001 C CNN "SPN"
-F 8 "-" H 0   0   50  0001 C CNN "SPURL"
+F 8 "https://www.digikey.com/products/en?keywords=296-37677-1-ND" H 0   0   50  0001 C CNN "SPURL"
 F 9 "IC REG BOOST ADJ 5.25A 16WQFN" H 0   0   50  0001 C CNN "DESC"
 	1    4950 3000
@@
 F 6 "Digikey" H 0   0   50  0001 C CNN "SPR"
 F 7 "541-2567-1-ND" H 0   0   50  0001 C CNN "SPN"
-F 8 "-" H 0   0   50  0001 C CNN "SPURL"
+F 8 "https://www.digikey.com/products/en?keywords=541-2567-1-ND" H 0   0   50  0001 C CNN "SPURL"
 F 9 "FIXED IND 3.3UH 2.7A 61 MOHM SMD" H 0   0   50  0001 C CNN "DESC"
 	1    4950 1900
@@
 F 6 "Digikey" H 0   0   50  0001 C CNN "SPR"
 F 7 "SS24FLCT-ND" H 0   0   50  0001 C CNN "SPN"
-F 8 "-" H 0   0   50  0001 C CNN "SPURL"
+F 8 "https://www.digikey.com/products/en?keywords=SS24FLCT-ND" H 0   0   50  0001 C CNN "SPURL"
 F 9 "DIODE SCHOTTKY 40V 2A SOD123F" H 0   0   50  0001 C CNN "DESC"
 	1    6300 2450
@@
 F 6 "Digikey" H 0   0   50  0001 C CNN "SPR"
 F 7 "490-11994-1-ND" H 0   0   50  0001 C CNN "SPN"
-F 8 "-" H 0   0   50  0001 C CNN "SPURL"
+F 8 "https://www.digikey.com/products/en?keywords=490-11994-1-ND" H 0   0   50  0001 C CNN "SPURL"
 F 9 "CAP CER 0.47UF 50V X5R 0603" H 0   0   50  0001 C CNN "DESC"
 	1    6400 3600
@@
 F 6 "Digikey" H 0   0   50  0001 C CNN "SPR"
 F 7 "541-2979-1-ND" H 0   0   50  0001 C CNN "SPN"
-F 8 "-" H 0   0   50  0001 C CNN "SPURL"
+F 8 "https://www.digikey.com/products/en?keywords=541-2979-1-ND" H 0   0   50  0001 C CNN "SPURL"
 F 9 "RES SMD 10K OHM 1% 1/10W 0603" H 0   0   50  0001 C CNN "DESC"
 	1    7100 3250
@@
 F 6 "Digikey" H 0   0   50  0001 C CNN "SPR"
 F 7 "541-86.6KHCT-ND" H 0   0   50  0001 C CNN "SPN"
-F 8 "-" H 0   0   50  0001 C CNN "SPURL"
+F 8 "https://www.digikey.com/products/en?keywords=541-86.6KHCT-ND" H 0   0   50  0001 C CNN "SPURL"
 F 9 "RES SMD 86.6K OHM 1% 1/10W 0603" H 0   0   50  0001 C CNN "DESC"
 	1    7100 2600
@@
 F 6 "Digikey" H 0   0   50  0001 C CNN "SPR"
 F 7 "1276-1946-1-ND" H 0   0   50  0001 C CNN "SPN"
-F 8 "-" H 0   0   50  0001 C CNN "SPURL"
+F 8 "https://www.digikey.com/products/en?keywords=1276-1946-1-ND" H 0   0   50  0001 C CNN "SPURL"
 F 9 "CAP CER 1UF 10V X7R 0603" H 0   0   50  0001 C CNN "DESC"
 	1    8000 2850
@@
 F 6 "Digikey" H 0   0   50  0001 C CNN "SPR"
 F 7 "490-4779-1-ND" H 0   0   50  0001 C CNN "SPN"
-F 8 "-" H 0   0   50  0001 C CNN "SPURL"
+F 8 "https://www.digikey.com/product-detail/en/murata-electronics/GCM188R71H104KA57D/490-4779-1-ND/1641698" H 0   0   50  0001 C CNN "SPURL"
 F 9 "CAP CER 0.1UF 50V X7R 0603" H 0   0   50  0001 C CNN "DESC"
 	1    3200 2750
 	1    0    0    -1
+$EndComp
+$Comp
+L Device:R R103
+U 1 1 5BAB141D
+P 6400 3300
+F 0 "R103" V 6193 3300 50  0000 C CNN
+F 1 "1.62K" V 6284 3300 50  0000 C CNN
+F 2 "Resistor_SMD:R_0603_1608Metric" V 6330 3300 50  0001 C CNN
+F 3 "https://www.yageo.com/upload/media/product/productsearch/datasheet/rchip/PYu-RC_Group_51_RoHS_L_10.pdf" H 6400 3300 50  0001 C CNN
+F 4 "Yageo" H 250 300 50  0001 C CNN "MFR"
+F 5 "RC0603FR-071K62L" H 250 300 50  0001 C CNN "MPN"
+F 6 "Digikey" H 250 300 50  0001 C CNN "SPR"
+F 7 "311-1.62KHRCT-ND" H 250 300 50  0001 C CNN "SPN"
+F 8 "https://www.digikey.com/product-detail/en/yageo/RC0603FR-071K62L/311-1.62KHRCT-ND/729816" H 250 300 50  0001 C CNN "SPURL"
+F 9 "RES SMD 1.62K OHM 1% 1/10W 0603" H 0   0   50  0001 C CNN "DESC"
+	1    6400 3300
+	-1   0    0    1
 $EndComp
 Text Label 5500 1900 0    50   ~ 0
@@
 Connection ~ 8900 3750
 NoConn ~ 5500 3900
-$Comp
-L Device:R R103
-U 1 1 5BAB141D
-P 6400 3300
-F 0 "R103" V 6193 3300 50  0000 C CNN
-F 1 "1.62K" V 6284 3300 50  0000 C CNN
-F 2 "Resistor_SMD:R_0603_1608Metric" V 6330 3300 50  0001 C CNN
-F 3 "https://www.yageo.com/upload/media/product/productsearch/datasheet/rchip/PYu-RC_Group_51_RoHS_L_10.pdf" H 6400 3300 50  0001 C CNN
-F 4 "Yageo" H 250 300 50  0001 C CNN "MFR"
-F 5 "RC0603FR-071K62L" H 250 300 50  0001 C CNN "MPN"
-F 6 "Digikey" H 250 300 50  0001 C CNN "SPR"
-F 7 "311-1.62KHRCT-ND" H 250 300 50  0001 C CNN "SPN"
-F 8 "https://www.digikey.com/product-detail/en/yageo/RC0603FR-071K62L/311-1.62KHRCT-ND/729816" H 250 300 50  0001 C CNN "SPURL"
-F 9 "RES SMD 1.62K OHM 1% 1/10W 0603" H 0   0   50  0001 C CNN "DESC"
-	1    6400 3300
-	-1   0    0    1
-$EndComp
 $EndSCHEMATC
