File: led-controller-wrover32/Reset_Boot.sch (KiCad schematic (older format))
At the start: 8 parts, among them Q5 BSS138DW-7-F, SW1 SW_SPST_KMR2, SW2 SW_SPST_KMR2

Commit message: Minor changes.
Signed-off-by: Aaron Williams <aaron.w2@gmail.com>
Parts:
- C5: MFR Samsung -> AVX; MPN CL10B104KO8WPNC -> 06035C104K4Z4A; SPN 1276-6582-1-ND -> 478-10679-1-ND
- R3: MFR (none) -> -; MPN (none) -> -; SPN (none) -> -; SPR (none) -> -; SPURL (none) -> -
- RN6: MFR Bourns -> Panasonic; MPN CAT16-1003F4LF -> EXB-V8V103JV; SPN CAT16-1003F4LFCT-ND -> Y4103CT-ND
